Commit message: pendulum differential drive

File: description/properties.xacro (robot description, xacro)
@@ -3,5 +3,5 @@
     <!-- Color Definitions -->
     <material name="white">
-        <color rgba= "1 1 1 1"/>
+        <color rgba= "1 1 1 0.5"/>
     </material>
     <material name="orange">

File: description/robot.urdf.xacro (robot description, xacro)
@@ -5,3 +5,5 @@
     <xacro:include filename="robot_core.xacro"/>
     <xacro:include filename="gazebo_control.xacro"/>
+    <xacro:include filename="lidar.xacro"/>
+    <xacro:include filename="imu.xacro"/>
 </robot>

File: description/robot_core.xacro (robot description, xacro)
@@ -9,23 +9,23 @@
         <parent link="base_link"/>
         <child link="chassis"/>
-        <origin xyz="-0.1 0 0"/>
+        <origin xyz="0 0 0.125"/>
     </joint>
     <!-- chassis link -->
     <link name="chassis">
         <visual>
-            <origin xyz="0.15 0 0.075"/>
+            <origin xyz="0.0 0.0 0.0"/>
             <geometry>
-                <box size="0.3 0.3 0.15"/>
+                <box size="0.1 0.3 0.25"/>
             </geometry>
             <material name="white"/>
         </visual>
         <collision>
-            <origin xyz="0.15 0 0.075"/>
+            <origin xyz="0.0 0.0 0.0"/>
             <geometry>
-                <box size="0.3 0.3 0.15"/>
+                <box size="0.1 0.3 0.25"/>
             </geometry>
         </collision>
-        <xacro:inertial_box mass="0.5" x="0.3" y="0.3" z="0.15">
-            <origin xyz="0.15 0 0.075" rpy="0 0 0"/>
+        <xacro:inertial_box mass="0.1" x="0.1" y="0.3" z="0.25">
+            <origin xyz="0.0 0.0 0.0" rpy="0 0 0"/>
         </xacro:inertial_box>
     </link>
@@ -78,27 +78,4 @@
         </xacro:inertial_cylinder>
     </link>
-    <!-- caster wheel joint -->
-    <joint name="caster_wheel_joint" type="fixed">
-        <parent link="chassis"/>
-        <child link="caster_wheel"/>
-        <origin xyz="0.24 0 0"/>
-    </joint>
-    <!-- left wheel link -->
-    <link name="caster_wheel">
-        <visual>
-            <geometry>
-                <sphere radius="0.05"/>
-            </geometry>
-            <material name="black"/>
-        </visual>
-        <collision>
-            <geometry>
-                <sphere radius="0.05"/>
-            </geometry>
-        </collision>
-        <xacro:inertial_sphere mass="0.1" radius="0.05">
-            <origin xyz="0 0 0" rpy="0 0 0"/>
-        </xacro:inertial_sphere>
-    </link>
     <gazebo reference="chassis">
         <material>Gazebo/White</material>
@@ -110,8 +87,3 @@
         <material>Gazebo/Blue</material>
     </gazebo>
-    <gazebo reference="caster_wheel">
-        <material>Gazebo/Black</material>
-        <mu1 value = "0.001" />
-        <mu2 value = "0.001" />
-    </gazebo>
 </robot>
